File: HARDWARE/Gringo/bpm-module.kicad_sch (KiCad schematic)
At the start: 21 parts, among them J17 Conn_01x05_Pin, U4 PTPS7A2018PDBVR, U5 MAX30101EFD+, U6 MAX32664GWEA+T, U7 PAM2401YPADJ, Y1 32k768

Commit message: Update the eval kit PCB and production files
Parts:
- renumbered C13 to C1, C15 to C2, C12 to C3, C14 to C4, C16 to C5, C17 to C6, C18 to C7
Changed lines of the file:
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@@
 		(dnp no)
 		(fields_autoplaced yes)
-		(property "Reference" "C18"
+		(property "Reference" "C7"
 			(at 207.01 126.9999 0)
 			(effects
@@
 			(project "Gringo"
 				(path "/d29665dc-a603-413d-b9b9-433aa1d50e1d/29d4f3f5-5c9e-40ce-940f-f091519cc096"
-					(reference "C18")
+					(reference "C7")
 					(unit 1)
 				)
@@
 		(on_board yes)
 		(dnp no)
-		(property "Reference" "C12"
+		(property "Reference" "C3"
 			(at 34.036 147.828 0)
 			(effects
@@
 			(project "Gringo"
 				(path "/d29665dc-a603-413d-b9b9-433aa1d50e1d/29d4f3f5-5c9e-40ce-940f-f091519cc096"
-					(reference "C12")
+					(reference "C3")
 					(unit 1)
 				)
@@
 		(on_board yes)
 		(dnp no)
-		(property "Reference" "C15"
+		(property "Reference" "C2"
 			(at 113.284 64.77 0)
 			(effects
@@
 			(project "Gringo"
 				(path "/d29665dc-a603-413d-b9b9-433aa1d50e1d/29d4f3f5-5c9e-40ce-940f-f091519cc096"
-					(reference "C15")
+					(reference "C2")
 					(unit 1)
 				)
@@
 		(on_board yes)
 		(dnp no)
-		(property "Reference" "C13"
+		(property "Reference" "C1"
 			(at 103.124 64.77 0)
 			(effects
@@
 			(project "Gringo"
 				(path "/d29665dc-a603-413d-b9b9-433aa1d50e1d/29d4f3f5-5c9e-40ce-940f-f091519cc096"
-					(reference "C13")
+					(reference "C1")
 					(unit 1)
 				)
@@
 		(on_board yes)
 		(dnp no)
-		(property "Reference" "C14"
+		(property "Reference" "C4"
 			(at 107.188 153.67 0)
 			(effects
@@
 			(project "Gringo"
 				(path "/d29665dc-a603-413d-b9b9-433aa1d50e1d/29d4f3f5-5c9e-40ce-940f-f091519cc096"
-					(reference "C14")
+					(reference "C4")
 					(unit 1)
 				)
@@
 		(on_board yes)
 		(dnp no)
-		(property "Reference" "C17"
+		(property "Reference" "C6"
 			(at 168.656 70.866 0)
 			(effects
@@
 			(project "Gringo"
 				(path "/d29665dc-a603-413d-b9b9-433aa1d50e1d/29d4f3f5-5c9e-40ce-940f-f091519cc096"
-					(reference "C17")
+					(reference "C6")
 					(unit 1)
 				)
@@
 		(on_board yes)
 		(dnp no)
-		(property "Reference" "C16"
+		(property "Reference" "C5"
 			(at 155.194 71.374 0)
 			(effects
@@
 			(project "Gringo"
 				(path "/d29665dc-a603-413d-b9b9-433aa1d50e1d/29d4f3f5-5c9e-40ce-940f-f091519cc096"
-					(reference "C16")
-					(unit 1)
-				)
+					(reference "C5")
+					(unit 1)
+				)

Commit message: Fix the evk board with the adapted component packages (#36)
* Correction before buy JLCPCB

Remove of via down to 2 tiny component
Change of clearance of the pads to pass routes
To remove clearance : select all the pads > propriétés > Clearance Overrides and DON T PUT 0 (herited) but something like -0.001

* Update scheme and PCB for evk boards with adapted component packages

* Update zones

* Update inductor package

* Update holes

* Update the quartz model

---------

Co-authored-by: bolobos <cartier.dc385@gmail.com>
Parts:
- removed U6: MAX32664GWEA+T, MAX32664GWEA-T:21-100241A_W161K1&plus_1_MXM, symbol MAX32664GWEA-functionnal:MAX32664GWEA+T
- added C8: 1u, Capacitor_SMD:C_0603_1608Metric, symbol Device:C
- added U8: MAX32664GTGA+T, MAX32664GTGA-T:21-100264_T2433&plus_2C_MXM, symbol MAX32664GTGA-T:MAX32664GTGA+T
- L1: footprint Inductor_SMD:L_0603_1608Metric -> Inductor_SMD:L_APV_ANR4030
- U5: footprint MAX30101EFD:21-1048_F143A5&plus_1_MXM-M -> MAX30101EFD-:21-1048_F143A5&plus_1_MXM
- Y1: footprint Crystal:Crystal_SMD_2012-2Pin_2.0x1.2mm -> ECS-327-12-5-12-TR:XTAL_ECX-12_2X1P2_ECS
- renumbered J17 to J13
Connections:
- net +1V8: now also C8.1, U8.11 (VDD), U8.22 (VDD)
- net GND: now also C8.2, U8.10 (VSS), U8.25 (EPAD), U8.7 (VSS)
- net HOST_SCL: now also U8.23 (SLAVE_SDA)
- net HOST_SDA: now also U8.24 (SLAVE_SCL)
- net HR_INT: now also U8.18 (HR_INT)
- net RST: now also U8.6 (RSTN)
- net SSR_SCL: now also U8.14 (SENSOR_SCL)
- net SSR_SDA: now also U8.13 (SENSOR_SDA)
- net at Y1.2: now also U8.8 (32KOUT)
- net at Y1.1: now also U8.9 (32KIN)
- net at C6.1: now also U8.12 (VCORE)
- no-connect marks 15 -> 12
