File: HARDWARE/Gringito/Gringito.kicad_sch (KiCad schematic)
At the start: 0 parts

Commit message: End schematics PCB Wireless Charge
Parts:
- added C1, C20: 0,01u, Capacitor_SMD:C_0805_2012Metric, symbol Device:C
- added C10, C15, C22, C26, C27, C3, C4, C8: 1u, Capacitor_SMD:C_0805_2012Metric, symbol Device:C
- added C11, C16, C18, C19, C21, C23, C24, C5, C6: 0,1u, Capacitor_SMD:C_0805_2012Metric, symbol Device:C
- added C12: 4,7n, Capacitor_SMD:C_0805_2012Metric, symbol Device:C
- added C13, C2, C25: 10u, Capacitor_SMD:C_0805_2012Metric, symbol Device:C
- added C14, C9: 4,7u, Capacitor_SMD:C_0805_2012Metric, symbol Device:C
- added C17: 4700p, Capacitor_SMD:C_0805_2012Metric, symbol Device:C
- added C7: 33p, Capacitor_SMD:C_0805_2012Metric, symbol Device:C
- added D1: LED, LED_SMD:LED_0805_2012Metric, symbol Device:LED
- added J1: USB_C_Receptacle_PowerOnly_6P, Connector_USB:USB_C_Receptacle_GCT_USB4135-GF-A_6P_TopMnt_Horizontal, symbol Connector:USB_C_Receptacle_PowerOnly_6P
- added J2: Conn_01x02, Connector_PinHeader_2.54mm:PinHeader_1x02_P2.54mm_Vertical, symbol Connector_Generic:Conn_01x02
- added L1: L, Connector_Wire:SolderWire-1.5sqmm_1x02_P6mm_D1.7mm_OD3mm, symbol Device:L
- added NT1: NetTie_2, NetTie:NetTie-2_SMD_Pad0.5mm, symbol Device:NetTie_2
- added R1: 1K, Resistor_SMD:R_0805_2012Metric_Pad1.20x1.40mm_HandSolder, symbol Device:R
- added R10, R5: 10R, Resistor_SMD:R_0805_2012Metric_Pad1.20x1.40mm_HandSolder, symbol Device:R
- added R11: 100K, Resistor_SMD:R_0805_2012Metric_Pad1.20x1.40mm_HandSolder, symbol Device:R
- added R12: 76K8, Resistor_SMD:R_0805_2012Metric_Pad1.20x1.40mm_HandSolder, symbol Device:R
- added R13, R15, R18, R19: 56,2K, Resistor_SMD:R_0805_2012Metric_Pad1.20x1.40mm_HandSolder, symbol Device:R
- added R14, R16, R23, R8: 10K, Resistor_SMD:R_0805_2012Metric_Pad1.20x1.40mm_HandSolder, symbol Device:R
- added R17: NTC, Resistor_SMD:R_0805_2012Metric_Pad1.20x1.40mm_HandSolder, symbol Device:R
- added R2, R4: 1R, Resistor_SMD:R_0805_2012Metric_Pad1.20x1.40mm_HandSolder, symbol Device:R
- added R20: 56K2, Resistor_SMD:R_0805_2012Metric_Pad1.20x1.40mm_HandSolder, symbol Device:R
- added R21, R22: 3,6K, Resistor_SMD:R_0805_2012Metric_Pad1.20x1.40mm_HandSolder, symbol Device:R
- added R24: 470, Resistor_SMD:R_0805_2012Metric_Pad1.20x1.40mm_HandSolder, symbol Device:R
- added R3: 20m, Resistor_SMD:R_0805_2012Metric_Pad1.20x1.40mm_HandSolder, symbol Device:R
- added R6, R7: 5K1, Resistor_SMD:R_0805_2012Metric_Pad1.20x1.40mm_HandSolder, symbol Device:R
- added R9: 12k1, Resistor_SMD:R_0805_2012Metric_Pad1.20x1.40mm_HandSolder, symbol Device:R
- added U1: PTPS7A2033PDBVR, DBV0005A-IPC_A, symbol ul_PTPS7A2033PDBVR:PTPS7A2033PDBVR
- added U2: INA199A1DCKR, DCK0006A_N, symbol ul_INA199A1DCKR:INA199A1DCKR
- added U3, U5: CSD97376Q4M, DPC0008A, symbol ul_CSD97376Q4M:CSD97376Q4M
- added U4: BQ500212ARGZR, RGZ0048A, symbol BQ500212ARGZR:BQ500212ARGZR
Connections:
- new net: L1.1, U3.4 (VSW)
- new net: C12.1, C16.2, C18.2, C19.2, C21.2, L1.2
- new net: C12.2, R11.1
- new net: C7.2, R10.2, R11.2, R8.1, R9.1
- new net: C16.1, C18.1, C19.1, C21.1, U5.4 (VSW)
- new net: C23.2, R23.1, U4.5 (RESET_N)
- new net: R15.1, U4.15 (FOD_CAL)
- new net: R18.1, U4.16 (PMOD)
- new net: R19.1, U4.17 (FOD)
- new net: C20.2, R16.1, R17.2, U4.2 (T_SENSE)
- new net: C26.2, C27.2, U4.35 (BPCAP)
- new net: R20.2, U4.44 (LED_MODE)
- new net: C17.1, R12.2, R14.1, U4.46 (V_SENSE)
- new net: C11.1, U3.6 (BOOT_R)
- new net: C11.2, U3.7 (BOOT)
- new net: C24.1, U5.6 (BOOT_R)
- new net: C24.2, U5.7 (BOOT)
- new net: R1.1, U2.6 (OUT)
- new net: C6.2, R2.2, U2.4 (IN+)
- new net: J1.A5 (CC1), R7.2
- new net: J1.B5 (CC2), R6.2
- new net: D1.2 (A), R24.1
- new net: C6.1, R4.2, U2.5 (IN-)
- new net +3V3: C1.1, C10.2, C14.1, C15.1, C26.1, C4.1, C9.2, R16.2, R23.2, R9.2, U1.5 (OUT), U2.3 (V+), U4.33 (V33D), U4.34 (V33A), U4.45 (RESERVED)
- new net COMM+: R10.1, U4.37 (COMM_A+), U4.39 (COMM_B+)
- new net COMM-: R5.1, U4.38 (COMM_A-), U4.40 (COMM_B-)
- new net DPWM-1A: R21.2, U3.8 (PWM), U4.12 (PWM_A)
- new net DPWM-1B: R22.2, U4.13 (PWM_B), U5.8 (PWM)
- new net GND: C13.2, C2.2, C22.2, C25.2, C3.2, C8.2, J1.A12 (GND), J1.B12 (GND), J1.S1 (SHIELD), J2.1 (Pin_1), NT1.2, R6.1, R7.1, U3.3 (PGND), U3.9 (PGND), U5.3 (PGND), U5.9 (PGND)
- new net GNDA: C1.2, C10.1, C14.2, C15.2, C17.2, C20.1, C23.1, C27.1, C4.2, C5.2, C7.1, C9.1, D1.1 (K), NT1.1, R13.2, R14.2, R17.1, R20.1, R21.1, R22.1, R5.2, R8.2, U1.2 (GND), U2.1 (REF), U2.2 (GND), U4.1 (PEAK_DET), U4.31 (GND), U4.32 (GND), U4.36 (GND), U4.47 (GND), U4.48 (ADCREF), U4.49 (EP)
- new net I_SENSE: C5.1, R1.2, U4.42 (I_SENSE)
- new net LED_A: R24.2, U4.7 (LED_A)
- new net LOSS_THR: R13.1, R15.2, R18.2, R19.2, U4.43 (LOSS_THR)
- new net VBUS: C2.1, C22.1, C3.1, C8.1, J1.A9 (VBUS), J1.B9 (VBUS), J2.2 (Pin_2), R12.1, R2.1, R3.2, U1.1 (IN), U1.3 (EN), U3.1 (SKIP_N), U3.2 (VDD), U5.1 (SKIP_N), U5.2 (VDD)
- new net VIN_MOSFET: C13.1, C25.1, R3.1, R4.1, U3.5 (VIN), U5.5 (VIN)
- no-connect marks 0 -> 23
Other:
- added sheet Reception (recep.kicad_sch)
- note added: "Bloc BQ500212A (Cerveau)"
- note added: "Bloc MOSFET / Bobine (Puissance)"
- note added: "LDO ALIM 5V -> 3.3 V"
- note added: "Led et lien de masse"
- note added: "Mesure de courant"

Commit message: final version + bom
Parts:
- C16, C18, C19, C21: footprint Capacitor_SMD:C_0805_2012Metric -> Capacitor_SMD:C_1206_3216Metric_Pad1.33x1.80mm_HandSolder
Changed lines of the file:
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@@
 			)
 		)
-		(property "Footprint" "Capacitor_SMD:C_0805_2012Metric"
+		(property "Footprint" "Capacitor_SMD:C_1206_3216Metric_Pad1.33x1.80mm_HandSolder"
 			(at 267.97 108.2548 0)
 			(effects
@@
 			)
 		)
-		(property "Footprint" "Capacitor_SMD:C_0805_2012Metric"
+		(property "Footprint" "Capacitor_SMD:C_1206_3216Metric_Pad1.33x1.80mm_HandSolder"
 			(at 267.97 126.0348 0)
 			(effects
@@
 			)
 		)
-		(property "Footprint" "Capacitor_SMD:C_0805_2012Metric"
+		(property "Footprint" "Capacitor_SMD:C_1206_3216Metric_Pad1.33x1.80mm_HandSolder"
 			(at 267.97 117.1448 0)
 			(effects
@@
 			)
 		)
-		(property "Footprint" "Capacitor_SMD:C_0805_2012Metric"
+		(property "Footprint" "Capacitor_SMD:C_1206_3216Metric_Pad1.33x1.80mm_HandSolder"
 			(at 267.97 99.3648 0)
 			(effects
