File: HARDWARE/Gringo-ring/alim_part.kicad_sch (KiCad schematic)
At the start: 22 parts, among them J13 Conn_01x05_Pin, U4 PTPS7A2018PDBVR, U5 MAX30101EFD+, U7 PAM2401YPADJ, U8 MAX32664GTGA+T, Y1 32k768

Commit message: Commit new organization of files on KiCAD
Parts:
- removed U4: PTPS7A2018PDBVR, PTPS7A2018PDBVR:DBV0005A-IPC_A, symbol PTPS7A2018PDBVR:PTPS7A2018PDBVR
- removed U5: MAX30101EFD+, MAX30101EFD-:21-1048_F143A5&plus_1_MXM, symbol MAX30101EFD:MAX30101EFD+
- removed U7: PAM2401YPADJ, PAM2401YPADJ:SON12_U-DFN3030-12_DIO-M, symbol PAM2401YPADJ:PAM2401YPADJ
- removed U8: MAX32664GTGA+T, MAX32664GTGA-T:21-100264_T2433&plus_2C_MXM, symbol MAX32664GTGA-T:MAX32664GTGA+T
- added U11: PAM2401YPADJ, PAM2401YPADJ:SON12_U-DFN3030-12_DIO-M, symbol PAM2401YPADJ:PAM2401YPADJ
- added U12: MAX30101EFD+, MAX30101EFD-:21-1048_F143A5&plus_1_MXM, symbol MAX30101EFD:MAX30101EFD+
- added U13: MAX32664GTGA+T, MAX32664GTGA-T:21-100264_T2433&plus_2C_MXM, symbol MAX32664GTGA-T:MAX32664GTGA+T
- added U14: PTPS7A2018PDBVR, PTPS7A2018PDBVR:DBV0005A-IPC_A, symbol PTPS7A2018PDBVR:PTPS7A2018PDBVR
Connections:
- net +1V8: now also U12.11 (VDD), U13.11 (VDD), U13.22 (VDD), U14.5 (OUT)
- net +3.3V: now also U11.3 (EN), U11.4 (VIN), U14.1 (IN), U14.3 (EN)
- net +5V: now also U11.10 (OUT), U11.9 (OUT), U12.10 (VLED+), U12.9 (VLED+)
- net GND: now also U11.11 (PGND), U11.12 (PGND), U11.6 (AGND), U12.12 (GND), U12.4 (PGND), U13.10 (VSS), U13.25 (EPAD), U13.7 (VSS), U14.2 (GND)
- net HOST_SCL: now also U13.23 (SLAVE_SDA)
- net HOST_SDA: now also U13.24 (SLAVE_SCL)
- net HR_INT: now also U12.13 (*INT), U13.18 (HR_INT)
- net RST: now also U13.6 (RSTN)
- net SSR_SCL: now also U12.2 (SCL), U13.14 (SENSOR_SCL)
- net SSR_SDA: now also U12.3 (SDA), U13.13 (SENSOR_SDA)
- net at Y1.1: now also U13.9 (32KIN)
- net at Y1.2: now also U13.8 (32KOUT)
- net at C6.1: now also U13.12 (VCORE)
- net at L1.2: now also U11.1 (LX), U11.2 (LX)
- net at R4.1, R5.1: now also U11.7 (FB)
