File: HARDWARE/Gringo-ring/untitled.kicad_sch (KiCad schematic)
At the start: 0 parts

Commit message: Add of schematics pages
Parts:
- added M1: Motor_DC, symbol Motor:Motor_DC
- added U2: MAX32664GWEA+T, 21-100241A_W161K1+1_MXM, symbol ul_MAX32664GWEA-T:MAX32664GWEA+T
- added U3: BHI260AB, BHI260AB_BOS, symbol ul_BHI260AB:BHI260AB
- added U4: STTS22HTR, UDFN-6L_2X2X0P5_STM, symbol ul_STTS22HTR:STTS22HTR
- added U5: DRV2605LDGS, Package_SO:VSSOP-10_3x3mm_P0.5mm, symbol Driver_Haptic:DRV2605LDGS
Other:
- added sheet Untitled Sheet (CHANDIEU.kicad_sch)

Commit message: Commit new organization of files on KiCAD
Parts:
- added IC1: BQ25120AYFPR, BGA25C40P5X5_247X253X50, symbol BQ25120AYFPR:BQ25120AYFPR
- added U6: BQ51013BRHLR, RHL20_2P05X3P05, symbol ul_BQ51013BRHLR:BQ51013BRHLR
Other:
- removed sheet Untitled Sheet
